Commit message: orientated arm

File: description/xacro/urdf.xacro (robot description, xacro)
@@ -73,5 +73,5 @@
     <!-- Instantiate the Alpha -->
     <xacro:alpha_5 parent="${prefix}manipulator_mount_link" name="$(arg prefix)">
-    <origin xyz="0 0 0" rpy="0 0 0" />
+    <origin xyz="0 0 0" rpy="${pi} 0 0" />
     </xacro:alpha_5>
     <!-- Instantiate the BlueROV2 -->

Commit message: update frames

File: description/xacro/urdf.xacro (robot description, xacro)
@@ -3,5 +3,12 @@
   <xacro:macro name="bluerov2_heavy_alpha_urdf" params="prefix">
     <!-- Robot world origin -->
-    <link name="world"/>
+    <link name="world">
+        <visual>
+        <origin rpy="0 0 0" xyz="0 0 0"/>
+        <geometry>
+            <cylinder radius="0.06" length="0.09"/>
+        </geometry>
+        </visual>
+    </link>
     <link name="world_bottom"/>
     <joint name="world_bottom_joint" type="fixed">

Commit message: fixed ~/description bug

File: description/xacro/urdf.xacro (robot description, xacro)
@@ -2,5 +2,5 @@
 <robot xmlns:xacro="http://ros.org/wiki/xacro">
   <xacro:macro name="bluerov2_heavy_alpha_urdf" params="prefix">
-    <!-- Robot world origin -->
+    <!-- world origin -->
     <link name="world">
         <visual>
@@ -17,9 +17,10 @@
       <origin xyz="0.0 0.0 -6.0" rpy="0 0 0"/>
     </joint>
+    <!-- Robot body origin -->
     <link name="base_link"/>
     <joint name="world_joint" type="fixed">
       <child link="base_link" />
       <parent link="world" />
-      <origin xyz="0.0 0.0 -1.0" rpy="0 0 0"/>
+      <origin xyz="0.0 0.0 -2.0" rpy="0 0 0"/>
     </joint>
     <link name="${prefix}manipulator_mount_link">

Commit message: update docs.rst

File: description/xacro/urdf.xacro (robot description, xacro)
@@ -22,5 +22,5 @@
       <child link="base_link" />
       <parent link="world" />
-      <origin xyz="0.0 0.0 -1.0" rpy="0 0 0"/>
+      <origin xyz="0.0 0.0 -0.5" rpy="0 0 0"/>
     </joint>
     <link name="${prefix}manipulator_mount_link">

Commit message: update initial vehicle pose

File: description/xacro/urdf.xacro (robot description, xacro)
@@ -22,5 +22,5 @@
       <child link="base_link" />
       <parent link="world" />
-      <origin xyz="0.0 0.0 -0.5" rpy="0 0 0"/>
+      <origin xyz="0.0 0.0 0.0" rpy="0 0 0"/>
     </joint>
     <link name="${prefix}manipulator_mount_link">
