Commit message: simulate imu

File: description/blue/xacro/bluerov2/urdf.xacro (robot description, xacro)
@@ -2,5 +2,4 @@
 <robot xmlns:xacro="http://ros.org/wiki/xacro">
   <xacro:macro name="bluerov2_urdf" params="prefix">
-    <link name="${prefix}base_footprint" />
     <link name="${prefix}base_link">
       <inertial>
@@ -32,7 +31,10 @@
       </collision>
     </link>
+      <!-- Robot Footprint -->
+    <link name="${prefix}base_footprint" />
     <joint name="${prefix}base_footprint_joint" type="fixed">
-      <parent link="${prefix}base_footprint" />
-      <child link="${prefix}base_link" />
+      <child link="${prefix}base_footprint" />
+      <parent link="${prefix}base_link" />
+      <origin xyz="0.0 0.0 -10.0" rpy="0 0 0"/>
     </joint>
     <!-- Import camera macro -->

File: description/blue/xacro/bluerov2_heavy/urdf.xacro (robot description, xacro)
@@ -2,5 +2,4 @@
 <robot xmlns:xacro="http://ros.org/wiki/xacro">
   <xacro:macro name="bluerov2_heavy_urdf" params="prefix">
-    <link name="${prefix}base_footprint" />
     <link name="${prefix}base_link">
       <inertial>
@@ -32,7 +31,10 @@
       </collision>
     </link>
+      <!-- Robot Footprint -->
+    <link name="${prefix}base_footprint" />
     <joint name="${prefix}base_footprint_joint" type="fixed">
-      <parent link="${prefix}base_footprint" />
-      <child link="${prefix}base_link" />
+      <child link="${prefix}base_footprint" />
+      <parent link="${prefix}base_link" />
+      <origin xyz="0.0 0.0 -10.0" rpy="0 0 0"/>
     </joint>
     <!-- Import camera macro -->

File: description/blue/xacro/bluerov2_heavy_reach/urdf.xacro (robot description, xacro)
@@ -2,5 +2,4 @@
 <robot xmlns:xacro="http://ros.org/wiki/xacro">
   <xacro:macro name="bluerov2_heavy_reach_urdf" params="prefix">
-    <link name="${prefix}base_footprint" />
     <link name="${prefix}base_link">
       <inertial>
@@ -32,7 +31,10 @@
       </collision>
     </link>
+      <!-- Robot Footprint -->
+    <link name="${prefix}base_footprint" />
     <joint name="${prefix}base_footprint_joint" type="fixed">
-      <parent link="${prefix}base_footprint" />
-      <child link="${prefix}base_link" />
+      <child link="${prefix}base_footprint" />
+      <parent link="${prefix}base_link" />
+      <origin xyz="0.0 0.0 1.0" rpy="0 0 0"/>
     </joint>
     <!-- Import camera macro -->
@@ -67,4 +69,98 @@
       <origin rpy="0 0 0" xyz="-0.118 0.215 0.064" />
     </xacro:t200_urdf>
+<!-- Define intertial property macros  -->
+  <xacro:macro name="box_inertia" params="m w h d">
+    <inertial>
+      <origin xyz="0 0 0" rpy="${pi/2} 0 ${pi/2}"/>
+      <mass value="${m}"/>
+      <inertia ixx="${(m/12) * (h*h + d*d)}" ixy="0.0" ixz="0.0" iyy="${(m/12) * (w*w + d*d)}" iyz="0.0" izz="${(m/12) * (w*w + h*h)}"/>
+    </inertial>
+  </xacro:macro>
+<link name="imu_link">
+  <visual>
+    <geometry>
+      <box size="0.1 0.1 0.1"/>
+    </geometry>
+  </visual>
+  <collision>
+    <geometry>
+      <box size="0.1 0.1 0.1"/>
+    </geometry>
+  </collision>
+  <xacro:box_inertia m="0.1" w="0.1" d="0.1" h="0.1"/>
+</link>
+<joint name="imu_joint" type="fixed">
+  <parent link="${prefix}base_link"/>
+  <child link="imu_link"/>
+  <origin xyz="0 0 0.01"/>
+</joint>
+ <gazebo reference="imu_link">
+  <sensor name="imu_sensor" type="imu">
+   <plugin filename="libgazebo_ros_imu_sensor.so" name="imu_plugin">
+      <ros>
+        <namespace>/demo</namespace>
+        <remapping>~/out:=imu</remapping>
+      </ros>
+      <initial_orientation_as_reference>false</initial_orientation_as_reference>
+    </plugin>
+    <always_on>true</always_on>
+    <update_rate>100</update_rate>
+    <visualize>true</visualize>
+    <imu>
+      <angular_velocity>
+        <x>
+          <noise type="gaussian">
+            <mean>0.0</mean>
+            <stddev>2e-4</stddev>
+            <bias_mean>0.0000075</bias_mean>
+            <bias_stddev>0.0000008</bias_stddev>
+          </noise>
+        </x>
+        <y>
+          <noise type="gaussian">
+            <mean>0.0</mean>
+            <stddev>2e-4</stddev>
+            <bias_mean>0.0000075</bias_mean>
+            <bias_stddev>0.0000008</bias_stddev>
+          </noise>
+        </y>
+        <z>
+          <noise type="gaussian">
+            <mean>0.0</mean>
+            <stddev>2e-4</stddev>
+            <bias_mean>0.0000075</bias_mean>
+            <bias_stddev>0.0000008</bias_stddev>
+          </noise>
+        </z>
+      </angular_velocity>
+      <linear_acceleration>
+        <x>
+          <noise type="gaussian">
+            <mean>0.0</mean>
+            <stddev>1.7e-2</stddev>
+            <bias_mean>0.1</bias_mean>
+            <bias_stddev>0.001</bias_stddev>
+          </noise>
+        </x>
+        <y>
+          <noise type="gaussian">
+            <mean>0.0</mean>
+            <stddev>1.7e-2</stddev>
+            <bias_mean>0.1</bias_mean>
+            <bias_stddev>0.001</bias_stddev>
+          </noise>
+        </y>
+        <z>
+          <noise type="gaussian">
+            <mean>0.0</mean>
+            <stddev>1.7e-2</stddev>
+            <bias_mean>0.1</bias_mean>
+            <bias_stddev>0.001</bias_stddev>
+          </noise>
+        </z>
+      </linear_acceleration>
+    </imu>
+  </sensor>
+</gazebo>
   </xacro:macro>
 </robot>
