Commit message: structuring for uvms simulation

File: description/alpha/urdf/alpha_5.urdf.xacro (robot description, xacro)
@@ -19,5 +19,5 @@
             <visual>
                 <geometry>
-                    <mesh filename="package://ros2_control_reach_5/meshes/M3-INLINE.stl"/>
+                    <mesh filename="package://ros2_control_reach_5/alpha/meshes/M3-INLINE.stl"/>
                 </geometry>
                 <origin rpy="0 0 0" xyz="0 0 0"/>
@@ -44,5 +44,5 @@
             <visual>
                 <geometry>
-                    <mesh filename="package://ros2_control_reach_5/meshes/M2-1-1.stl"/>
+                    <mesh filename="package://ros2_control_reach_5/alpha/meshes/M2-1-1.stl"/>
                 </geometry>
                 <origin rpy="0 0 0" xyz="0 0 0"/>
@@ -71,5 +71,5 @@
             <visual>
                 <geometry>
-                    <mesh filename="package://ros2_control_reach_5/meshes/M2.stl"/>
+                    <mesh filename="package://ros2_control_reach_5/alpha/meshes/M2.stl"/>
                 </geometry>
                 <origin rpy="0 0 0" xyz="0 0 0"/>
@@ -110,5 +110,5 @@
             <visual>
                 <geometry>
-                    <mesh filename="package://ros2_control_reach_5/meshes/M2-1-3.stl"/>
+                    <mesh filename="package://ros2_control_reach_5/alpha/meshes/M2-1-3.stl"/>
                 </geometry>
                 <origin rpy="0 0 0" xyz="0 0 0"/>
@@ -137,5 +137,5 @@
             <visual>
                 <geometry>
-                    <mesh filename="package://ros2_control_reach_5/meshes/RS1-100-101-123.stl"/>
+                    <mesh filename="package://ros2_control_reach_5/alpha/meshes/RS1-100-101-123.stl"/>
                 </geometry>
                 <origin rpy="0 -1.5707 0" xyz="0 0 0"/>
@@ -174,5 +174,5 @@
             <limit effort="10" lower="0" upper="0.015" velocity="10"/>
         </joint>
-        <xacro:include filename="$(find ros2_control_reach_5)/urdf/end_effectors/standard_jaws.urdf.xacro"/>
+        <xacro:include filename="$(find ros2_control_reach_5)/alpha/urdf/end_effectors/standard_jaws.urdf.xacro"/>
         <xacro:alpha_standard_jaws parent="${name}_jaws_base_link" name="${name}_standard_jaws" axis_a="${name}_axis_a">
             <origin xyz="0 0 0" rpy="0 0 0"/>

File: description/alpha/urdf/end_effectors/standard_jaws.urdf.xacro (robot description, xacro)
@@ -14,5 +14,5 @@
             <visual>
                 <geometry>
-                    <mesh filename="package://ros2_control_reach_5/meshes/end_effectors/RS1-124.stl"/>
+                    <mesh filename="package://ros2_control_reach_5/alpha/meshes/end_effectors/RS1-124.stl"/>
                 </geometry>
                 <material name="${name}_black"/>
@@ -22,5 +22,5 @@
             <visual>
                 <geometry>
-                    <mesh filename="package://ros2_control_reach_5/meshes/end_effectors/RS1-130.stl"/>
+                    <mesh filename="package://ros2_control_reach_5/alpha/meshes/end_effectors/RS1-130.stl"/>
                 </geometry>
                 <material name="${name}_black"/>
@@ -45,5 +45,5 @@
             <visual>
                 <geometry>
-                    <mesh filename="package://ros2_control_reach_5/meshes/end_effectors/RS1-139.stl"/>
+                    <mesh filename="package://ros2_control_reach_5/alpha/meshes/end_effectors/RS1-139.stl"/>
                 </geometry>
                 <material name="${name}_black"/>

File: description/xacro/robot_system_multi_interface.urdf.xacro (robot description, xacro)
@@ -13,5 +13,5 @@
   <xacro:arg name="state_update_frequency" default="250"/>
   <!-- Import RRBot macro -->
-  <xacro:include filename="$(find ros2_control_reach_5)/urdf/alpha_5.urdf.xacro"/>
+  <xacro:include filename="$(find ros2_control_reach_5)/alpha/urdf/alpha_5.urdf.xacro"/>
   <!-- Import RRBot ros2_control description -->
   <xacro:include filename="$(find ros2_control_reach_5)/ros2_control/robot_system_multi_interface.ros2_control.xacro" />

Commit message: state and comms for blue in ros2_control added

File: description/alpha/urdf/alpha_5.urdf.xacro (robot description, xacro)
@@ -19,5 +19,5 @@
             <visual>
                 <geometry>
-                    <mesh filename="package://ros2_control_reach_5/alpha/meshes/M3-INLINE.stl"/>
+                    <mesh filename="package://ros2_control_blue_reach_5/alpha/meshes/M3-INLINE.stl"/>
                 </geometry>
                 <origin rpy="0 0 0" xyz="0 0 0"/>
@@ -44,5 +44,5 @@
             <visual>
                 <geometry>
-                    <mesh filename="package://ros2_control_reach_5/alpha/meshes/M2-1-1.stl"/>
+                    <mesh filename="package://ros2_control_blue_reach_5/alpha/meshes/M2-1-1.stl"/>
                 </geometry>
                 <origin rpy="0 0 0" xyz="0 0 0"/>
@@ -71,5 +71,5 @@
             <visual>
                 <geometry>
-                    <mesh filename="package://ros2_control_reach_5/alpha/meshes/M2.stl"/>
+                    <mesh filename="package://ros2_control_blue_reach_5/alpha/meshes/M2.stl"/>
                 </geometry>
                 <origin rpy="0 0 0" xyz="0 0 0"/>
@@ -110,5 +110,5 @@
             <visual>
                 <geometry>
-                    <mesh filename="package://ros2_control_reach_5/alpha/meshes/M2-1-3.stl"/>
+                    <mesh filename="package://ros2_control_blue_reach_5/alpha/meshes/M2-1-3.stl"/>
                 </geometry>
                 <origin rpy="0 0 0" xyz="0 0 0"/>
@@ -137,5 +137,5 @@
             <visual>
                 <geometry>
-                    <mesh filename="package://ros2_control_reach_5/alpha/meshes/RS1-100-101-123.stl"/>
+                    <mesh filename="package://ros2_control_blue_reach_5/alpha/meshes/RS1-100-101-123.stl"/>
                 </geometry>
                 <origin rpy="0 -1.5707 0" xyz="0 0 0"/>
@@ -174,5 +174,5 @@
             <limit effort="10" lower="0" upper="0.015" velocity="10"/>
         </joint>
-        <xacro:include filename="$(find ros2_control_reach_5)/alpha/urdf/end_effectors/standard_jaws.urdf.xacro"/>
+        <xacro:include filename="$(find ros2_control_blue_reach_5)/alpha/urdf/end_effectors/standard_jaws.urdf.xacro"/>
         <xacro:alpha_standard_jaws parent="${name}_jaws_base_link" name="${name}_standard_jaws" axis_a="${name}_axis_a">
             <origin xyz="0 0 0" rpy="0 0 0"/>

File: description/alpha/urdf/end_effectors/standard_jaws.urdf.xacro (robot description, xacro)
@@ -14,5 +14,5 @@
             <visual>
                 <geometry>
-                    <mesh filename="package://ros2_control_reach_5/alpha/meshes/end_effectors/RS1-124.stl"/>
+                    <mesh filename="package://ros2_control_blue_reach_5/alpha/meshes/end_effectors/RS1-124.stl"/>
                 </geometry>
                 <material name="${name}_black"/>
@@ -22,5 +22,5 @@
             <visual>
                 <geometry>
-                    <mesh filename="package://ros2_control_reach_5/alpha/meshes/end_effectors/RS1-130.stl"/>
+                    <mesh filename="package://ros2_control_blue_reach_5/alpha/meshes/end_effectors/RS1-130.stl"/>
                 </geometry>
                 <material name="${name}_black"/>
@@ -45,5 +45,5 @@
             <visual>
                 <geometry>
-                    <mesh filename="package://ros2_control_reach_5/alpha/meshes/end_effectors/RS1-139.stl"/>
+                    <mesh filename="package://ros2_control_blue_reach_5/alpha/meshes/end_effectors/RS1-139.stl"/>
                 </geometry>
                 <material name="${name}_black"/>

File: description/blue/xacro/bluerov2/urdf.xacro (robot description, xacro)
@@ -19,5 +19,5 @@
         <geometry>
           <mesh
-            filename="package://ros2_control_reach_5/blue/meshes/bluerov2/bluerov2.dae"
+            filename="package://ros2_control_blue_reach_5/blue/meshes/bluerov2/bluerov2.dae"
             scale="0.025 0.025 0.025"
           />
@@ -37,10 +37,10 @@
     </joint>
     <!-- Import camera macro -->
-    <xacro:include filename="$(find ros2_control_reach_5)/blue/xacro/camera/urdf.xacro" />
+    <xacro:include filename="$(find ros2_control_blue_reach_5)/blue/xacro/camera/urdf.xacro" />
     <xacro:camera_urdf prefix="${prefix}" parent="${prefix}base_link">
       <origin rpy="0 0 0" xyz="0.21 0 0.067" />
     </xacro:camera_urdf>
     <!-- Import T200 macro -->
-    <xacro:include filename="$(find ros2_control_reach_5)/blue/xacro/t200/urdf.xacro" />
+    <xacro:include filename="$(find ros2_control_blue_reach_5)/blue/xacro/t200/urdf.xacro" />
     <xacro:t200_urdf parent="${prefix}base_link" prefix="${prefix}" ccw="true" id="1">
       <origin rpy="-1.571 1.571 -0.785" xyz="0.14 -0.092 0.0" />

File: description/blue/xacro/bluerov2_heavy/urdf.xacro (robot description, xacro)
@@ -19,5 +19,5 @@
         <geometry>
           <mesh
-            filename="package://ros2_control_reach_5/blue/meshes/bluerov2_heavy/bluerov2_heavy.dae"
+            filename="package://ros2_control_blue_reach_5/blue/meshes/bluerov2_heavy/bluerov2_heavy.dae"
             scale="0.025 0.025 0.025"
           />
@@ -37,10 +37,10 @@
     </joint>
     <!-- Import camera macro -->
-    <xacro:include filename="$(find ros2_control_reach_5)/blue/xacro/camera/urdf.xacro" />
+    <xacro:include filename="$(find ros2_control_blue_reach_5)/blue/xacro/camera/urdf.xacro" />
     <xacro:camera_urdf prefix="${prefix}" parent="${prefix}base_link">
       <origin rpy="0 0 0" xyz="0.21 0 0.067" />
     </xacro:camera_urdf>
     <!-- Import T200 macro -->
-    <xacro:include filename="$(find ros2_control_reach_5)/blue/xacro/t200/urdf.xacro" />
+    <xacro:include filename="$(find ros2_control_blue_reach_5)/blue/xacro/t200/urdf.xacro" />
     <xacro:t200_urdf parent="${prefix}base_link" prefix="${prefix}" ccw="true" id="1">
       <origin rpy="-1.571 1.571 -0.785" xyz="0.14 -0.092 0.0" />

File: description/blue/xacro/bluerov2_heavy_reach/urdf.xacro (robot description, xacro)
@@ -19,5 +19,5 @@
         <geometry>
           <mesh
-            filename="package://ros2_control_reach_5/blue/meshes/bluerov2_heavy_reach/bluerov2_heavy_reach.dae"
+            filename="package://ros2_control_blue_reach_5/blue/meshes/bluerov2_heavy_reach/bluerov2_heavy_reach.dae"
             scale="0.025 0.025 0.025"
           />
@@ -37,10 +37,10 @@
     </joint>
     <!-- Import camera macro -->
-    <xacro:include filename="$(find ros2_control_reach_5)/blue/xacro/camera/urdf.xacro" />
+    <xacro:include filename="$(find ros2_control_blue_reach_5)/blue/xacro/camera/urdf.xacro" />
     <xacro:camera_urdf prefix="${prefix}" parent="${prefix}base_link">
       <origin rpy="0 0 0" xyz="0.21 0 0.067" />
     </xacro:camera_urdf>
     <!-- Import T200 macro -->
-    <xacro:include filename="$(find ros2_control_reach_5)/blue/xacro/t200/urdf.xacro" />
+    <xacro:include filename="$(find ros2_control_blue_reach_5)/blue/xacro/t200/urdf.xacro" />
     <xacro:t200_urdf parent="${prefix}base_link" prefix="${prefix}" ccw="true" id="1">
       <origin rpy="-1.571 1.571 -1.047" xyz="0.088 -0.102 -0.04" />

File: description/blue/xacro/t200/urdf.xacro (robot description, xacro)
@@ -17,10 +17,10 @@
         <xacro:if value="${ccw}">
           <geometry>
-            <mesh filename="package://ros2_control_reach_5/blue/meshes/t200/ccw_prop.dae" />
+            <mesh filename="package://ros2_control_blue_reach_5/blue/meshes/t200/ccw_prop.dae" />
           </geometry>
         </xacro:if>
         <xacro:unless value="${ccw}">
           <geometry>
-            <mesh filename="package://ros2_control_reach_5/blue/meshes/t200/cw_prop.dae" />
+            <mesh filename="package://ros2_control_blue_reach_5/blue/meshes/t200/cw_prop.dae" />
           </geometry>
         </xacro:unless>

File: description/ros2_control/robot_system_multi_interface.ros2_control.xacro (robot description, xacro)
@@ -6,5 +6,5 @@
       <hardware>
         <xacro:if value="${use_mock_hardware}">
-          <plugin>ros2_control_reach_5/RRBotSystemMultiInterfaceHardware</plugin>
+          <plugin>ros2_control_blue_reach_5/RRBotSystemMultiInterfaceHardware</plugin>
           <param name="example_param_hw_start_duration_sec">0.0</param>
           <param name="example_param_hw_stop_duration_sec">3.0</param>
@@ -12,5 +12,5 @@
         </xacro:if>
         <xacro:unless value="${use_mock_hardware}">
-          <plugin>ros2_control_reach_5/ReachSystemMultiInterfaceHardware</plugin>
+          <plugin>ros2_control_blue_reach_5/ReachSystemMultiInterfaceHardware</plugin>
           <param name="serial_port">${serial_port}</param>
           <param name="state_update_frequency">${state_update_frequency}</param>

File: description/xacro/robot_system_multi_interface.urdf.xacro (robot description, xacro)
@@ -8,5 +8,5 @@
   <xacro:arg name="state_update_frequency" default="250"/>
     <!-- Properties -->
-  <xacro:property name="description_package" value="ros2_control_reach_5" />
+  <xacro:property name="description_package" value="ros2_control_blue_reach_5" />
   <xacro:property name="prefix" value="$(arg prefix)" />
   <!-- Imports -->
@@ -14,4 +14,6 @@
   <!-- Import RRBot ros2_control description -->
   <xacro:include filename="$(find ${description_package})/ros2_control/robot_system_multi_interface.ros2_control.xacro" />
+  <!-- Import RRBot ros2_control description -->
+  <xacro:include filename="$(find ${description_package})/ros2_control/vehicle_system_multi_interface.ros2_control.xacro" />
   <xacro:bluerov2_heavy_alpha_urdf
     prefix="${prefix}" />
@@ -23,3 +25,10 @@
     use_mock_hardware="$(arg use_mock_hardware)"
     slowdown="$(arg slowdown)" />
+  <xacro:vehicle_system_multi_interface
+    name="BlueSystemMultiInterface"
+    prefix="$(arg prefix)"
+    serial_port="$(arg serial_port)"
+    state_update_frequency="$(arg state_update_frequency)"
+    use_mock_hardware="$(arg use_mock_hardware)"
+    slowdown="$(arg slowdown)" />
 </robot>

File: description/xacro/urdf.xacro (robot description, xacro)
@@ -69,6 +69,6 @@
     </joint>
     <!-- Imports -->
-    <xacro:include filename="$(find ros2_control_reach_5)/alpha/urdf/alpha_5.urdf.xacro" />
-    <xacro:include filename="$(find ros2_control_reach_5)/blue/xacro/bluerov2_heavy_reach/urdf.xacro" />
+    <xacro:include filename="$(find ros2_control_blue_reach_5)/alpha/urdf/alpha_5.urdf.xacro" />
+    <xacro:include filename="$(find ros2_control_blue_reach_5)/blue/xacro/bluerov2_heavy_reach/urdf.xacro" />
     <!-- Instantiate the Alpha -->
     <xacro:alpha_5 parent="${prefix}manipulator_mount_link" name="$(arg prefix)">

Commit message: testing controller

File: description/alpha/urdf/alpha_5.urdf.xacro (robot description, xacro)
@@ -15,5 +15,5 @@
                 <origin xyz="-75e-3 -6e-3 -3e-3" rpy="0 0 0"/>
                 <mass value="0.341"/>
-                <inertia ixx="83.66e-6"  ixy="14.45e-6"  ixz="-38.270e-6" iyy="998.81e-6" iyz="3.14e-6" izz="1003.60e-6" />
+                <inertia ixx="83.66e-6"  ixy="0.0"  ixz="0.0" iyy="998.81e-6" iyz="0.0" izz="1003.60e-6" />
             </inertial>
             <visual>
@@ -38,7 +38,7 @@
         <link name="${name}_m2_1_1_link">
             <inertial>
-                <origin xyz="0.042 0.009 0.142" rpy="0 0 0"/>
+                <origin xyz="5e-3 -1e-3 16e-3" rpy="0 0 0"/>
                 <mass value="0.194"/>
-                <inertia ixx="8.000"  ixy="-0.283"  ixz="0.289" iyy="7.922" iyz="0.074" izz="0.318" />
+                <inertia ixx="139.140e-6"  ixy="0.0"  ixz="0.0" iyy="158.490e-6" iyz="0.0" izz="61.960e-6" />
             </inertial>
             <visual>
@@ -65,7 +65,7 @@
         <link name="${name}_m2_joint_link">
             <inertial>
-                <origin xyz="0.013 -0.003 -0.021" rpy="0 0 0"/>
+                <origin xyz="73.563e-3 -0.091e-3 -0.734e-3" rpy="0 0 0"/>
                 <mass value="0.429"/>
-                <inertia ixx="0.795"  ixy="-2.240"  ixz="0.412" iyy="0.574" iyz="-0.359" izz="0.511" />
+                <inertia ixx="86.770e-6"  ixy="0.0"  ixz="0.0" iyy="868.230e-6" iyz="0.0" izz="891.460e-6" />
             </inertial>
             <visual>
@@ -104,7 +104,7 @@
         <link name="${name}_m2_1_2_link">
             <inertial>
-                <origin xyz="0.027 0.034 0.030" rpy="0 0 0"/>
+                <origin xyz="17e-3 -26e-3 2e-3" rpy="0 0 0"/>
                 <mass value="0.115"/>
-                <inertia ixx="0.529"  ixy="-0.899"  ixz="-0.072" iyy="0.255" iyz="-0.064" izz="0.692" />
+                <inertia ixx="41.800e-6"  ixy="0.0"  ixz="0.0" iyy="28.300e-6" iyz="0.0" izz="45.020e-6" />
             </inertial>
             <visual>
@@ -131,7 +131,7 @@
         <link name="${name}_m1_link">
             <inertial>
-                <origin xyz="-0.027 0.006 -0.004" rpy="0 0 0"/>
+                <origin xyz="-0.030e-3 -3.000e-3 -98.00e-3" rpy="0 0 0"/>
                 <mass value="0.333"/>
-                <inertia ixx="0.268"  ixy="-0.144"  ixz="0.049" iyy="0.387" iyz="-0.211" izz="0.260" />
+                <inertia ixx="507.870e-6"  ixy="0.0"  ixz="0.0" iyy="535.870e-6" iyz="0.0" izz="76.000e-6" />
             </inertial>
             <visual>

Commit message: updates

File: description/alpha/urdf/alpha_5.urdf.xacro (robot description, xacro)
@@ -19,5 +19,5 @@
             <visual>
                 <geometry>
-                    <mesh filename="package://ros2_control_blue_reach_5/alpha/meshes/M3-INLINE.stl"/>
+                    <mesh filename="file://$(find ros2_control_blue_reach_5)/alpha/meshes/M3-INLINE.stl"/>
                 </geometry>
                 <origin rpy="0 0 0" xyz="0 0 0"/>
@@ -44,5 +44,5 @@
             <visual>
                 <geometry>
-                    <mesh filename="package://ros2_control_blue_reach_5/alpha/meshes/M2-1-1.stl"/>
+                    <mesh filename="file://$(find ros2_control_blue_reach_5)/alpha/meshes/M2-1-1.stl"/>
                 </geometry>
                 <origin rpy="0 0 0" xyz="0 0 0"/>
@@ -71,5 +71,5 @@
             <visual>
                 <geometry>
-                    <mesh filename="package://ros2_control_blue_reach_5/alpha/meshes/M2.stl"/>
+                    <mesh filename="file://$(find ros2_control_blue_reach_5)/alpha/meshes/M2.stl"/>
                 </geometry>
                 <origin rpy="0 0 0" xyz="0 0 0"/>
@@ -110,5 +110,5 @@
             <visual>
                 <geometry>
-                    <mesh filename="package://ros2_control_blue_reach_5/alpha/meshes/M2-1-3.stl"/>
+                    <mesh filename="file://$(find ros2_control_blue_reach_5)/alpha/meshes/M2-1-3.stl"/>
                 </geometry>
                 <origin rpy="0 0 0" xyz="0 0 0"/>
@@ -137,5 +137,5 @@
             <visual>
                 <geometry>
-                    <mesh filename="package://ros2_control_blue_reach_5/alpha/meshes/RS1-100-101-123.stl"/>
+                    <mesh filename="file://$(find ros2_control_blue_reach_5)/alpha/meshes/RS1-100-101-123.stl"/>
                 </geometry>
                 <origin rpy="0 -1.5707 0" xyz="0 0 0"/>

File: description/alpha/urdf/end_effectors/standard_jaws.urdf.xacro (robot description, xacro)
@@ -14,5 +14,5 @@
             <visual>
                 <geometry>
-                    <mesh filename="package://ros2_control_blue_reach_5/alpha/meshes/end_effectors/RS1-124.stl"/>
+                    <mesh filename="file://$(find ros2_control_blue_reach_5)/alpha/meshes/end_effectors/RS1-124.stl"/>
                 </geometry>
                 <material name="${name}_black"/>
@@ -22,5 +22,5 @@
             <visual>
                 <geometry>
-                    <mesh filename="package://ros2_control_blue_reach_5/alpha/meshes/end_effectors/RS1-130.stl"/>
+                    <mesh filename="file://$(find ros2_control_blue_reach_5)/alpha/meshes/end_effectors/RS1-130.stl"/>
                 </geometry>
                 <material name="${name}_black"/>
@@ -45,5 +45,5 @@
             <visual>
                 <geometry>
-                    <mesh filename="package://ros2_control_blue_reach_5/alpha/meshes/end_effectors/RS1-139.stl"/>
+                    <mesh filename="file://$(find ros2_control_blue_reach_5)/alpha/meshes/end_effectors/RS1-139.stl"/>
                 </geometry>
                 <material name="${name}_black"/>

File: description/blue/xacro/bluerov2_heavy_reach/urdf.xacro (robot description, xacro)
@@ -18,5 +18,5 @@
         <geometry>
           <mesh
-            filename="package://ros2_control_blue_reach_5/blue/meshes/bluerov2_heavy_reach/bluerov2_heavy_reach.dae"
+            filename="file://$(find ros2_control_blue_reach_5)/blue/meshes/bluerov2_heavy_reach/bluerov2_heavy_reach.dae"
             scale="0.025 0.025 0.025"
           />

File: description/blue/xacro/t200/urdf.xacro (robot description, xacro)
@@ -17,10 +17,10 @@
         <xacro:if value="${ccw}">
           <geometry>
-            <mesh filename="package://ros2_control_blue_reach_5/blue/meshes/t200/ccw_prop.dae" />
+            <mesh filename="file://$(find ros2_control_blue_reach_5)/blue/meshes/t200/ccw_prop.dae" />
           </geometry>
         </xacro:if>
         <xacro:unless value="${ccw}">
           <geometry>
-            <mesh filename="package://ros2_control_blue_reach_5/blue/meshes/t200/cw_prop.dae" />
+            <mesh filename="file://$(find ros2_control_blue_reach_5)/blue/meshes/t200/cw_prop.dae" />
           </geometry>
         </xacro:unless>
