Commit message: update

File: description/blue/xacro/bluerov2_heavy_reach/urdf.xacro (robot description, xacro)
@@ -70,9 +70,9 @@
     </xacro:t200_urdf>
 <!-- Define intertial property macros  -->
-  <xacro:macro name="box_inertia" params="m w h d">
+  <xacro:macro name="box_inertia">
     <inertial>
       <origin xyz="0 0 0" rpy="${pi/2} 0 ${pi/2}"/>
-      <mass value="${m}"/>
-      <inertia ixx="${(m/12) * (h*h + d*d)}" ixy="0.0" ixz="0.0" iyy="${(m/12) * (w*w + d*d)}" iyz="0.0" izz="${(m/12) * (w*w + h*h)}"/>
+      <mass value="0.0"/>
+      <inertia ixx="0.0" ixy="0.0" ixz="0.0" iyy="0.0" iyz="0.0" izz="0.0"/>
     </inertial>
   </xacro:macro>
@@ -80,13 +80,13 @@
   <visual>
     <geometry>
-      <box size="0.1 0.1 0.1"/>
+      <box size="0.01 0.01 0.01"/>
     </geometry>
   </visual>
   <collision>
     <geometry>
-      <box size="0.1 0.1 0.1"/>
+      <box size="0.01 0.01 0.01"/>
     </geometry>
   </collision>
-  <xacro:box_inertia m="0.1" w="0.1" d="0.1" h="0.1"/>
+  <xacro:box_inertia/>
 </link>
 <joint name="imu_joint" type="fixed">

File: description/ros2_control/robot_system_multi_interface.ros2_control.xacro (robot description, xacro)
@@ -49,4 +49,5 @@
         <state_interface name="acceleration"/>
         <state_interface name="current"/>
+        <state_interface name="stateId"/>
       </joint>
       <joint name="${prefix}_axis_b">
@@ -80,4 +81,5 @@
         <state_interface name="acceleration"/>
         <state_interface name="current"/>
+        <state_interface name="stateId"/>
       </joint>
       <joint name="${prefix}_axis_c">
@@ -111,4 +113,5 @@
         <state_interface name="acceleration"/>
         <state_interface name="current"/>
+        <state_interface name="stateId"/>
       </joint>
       <joint name="${prefix}_axis_d">
@@ -142,4 +145,5 @@
         <state_interface name="acceleration"/>
         <state_interface name="current"/>
+        <state_interface name="stateId"/>
       </joint>
       <joint name="${prefix}_axis_e">
@@ -173,4 +177,5 @@
         <state_interface name="acceleration"/>
         <state_interface name="current"/>
+        <state_interface name="stateId"/>
       </joint>
     </ros2_control>

File: description/xacro/robot_system_multi_interface.urdf.xacro (robot description, xacro)
@@ -12,4 +12,5 @@
   <!-- Imports -->
  <xacro:include filename="$(find ${description_package})/xacro/urdf.xacro"/>
+  <!-- <xacro:include filename="$(find ${description_package})/blue/xacro/bluerov2_heavy_reach/urdf.xacro"/> -->
   <!-- Import RRBot ros2_control description -->
   <xacro:include filename="$(find ${description_package})/ros2_control/robot_system_multi_interface.ros2_control.xacro" />

File: description/xacro/urdf.xacro (robot description, xacro)
@@ -2,5 +2,5 @@
 <robot xmlns:xacro="http://ros.org/wiki/xacro">
   <xacro:macro name="bluerov2_heavy_alpha_urdf" params="prefix">
-    <!-- <link name="${prefix}base_link"/> -->
+    <link name="base_link"/>
     <link name="${prefix}manipulator_mount_link">
       <visual>
@@ -58,4 +58,9 @@
       </collision>
     </link>
+    <joint name="${prefix}base_joint" type="fixed">
+      <child link="${prefix}base_link" />
+      <parent link="base_link" />
+      <origin xyz="0.0 0.0 0.0" rpy="0 0 0"/>
+    </joint>
     <joint name="${prefix}manipulator_mount_joint" type="fixed">
       <origin rpy="0 0 0" xyz="0.14 0.0 -0.12" />

Commit message: dynamics revision

File: description/blue/xacro/bluerov2_heavy_reach/urdf.xacro (robot description, xacro)
@@ -69,98 +69,4 @@
       <origin rpy="0 0 0" xyz="-0.118 0.215 0.064" />
     </xacro:t200_urdf>
-<!-- Define intertial property macros  -->
-  <xacro:macro name="box_inertia">
-    <inertial>
-      <origin xyz="0 0 0" rpy="${pi/2} 0 ${pi/2}"/>
-      <mass value="0.0"/>
-      <inertia ixx="0.0" ixy="0.0" ixz="0.0" iyy="0.0" iyz="0.0" izz="0.0"/>
-    </inertial>
-  </xacro:macro>
-<link name="imu_link">
-  <visual>
-    <geometry>
-      <box size="0.01 0.01 0.01"/>
-    </geometry>
-  </visual>
-  <collision>
-    <geometry>
-      <box size="0.01 0.01 0.01"/>
-    </geometry>
-  </collision>
-  <xacro:box_inertia/>
-</link>
-<joint name="imu_joint" type="fixed">
-  <parent link="${prefix}base_link"/>
-  <child link="imu_link"/>
-  <origin xyz="0 0 0.01"/>
-</joint>
- <gazebo reference="imu_link">
-  <sensor name="imu_sensor" type="imu">
-   <plugin filename="libgazebo_ros_imu_sensor.so" name="imu_plugin">
-      <ros>
-        <namespace>/demo</namespace>
-        <remapping>~/out:=imu</remapping>
-      </ros>
-      <initial_orientation_as_reference>false</initial_orientation_as_reference>
-    </plugin>
-    <always_on>true</always_on>
-    <update_rate>100</update_rate>
-    <visualize>true</visualize>
-    <imu>
-      <angular_velocity>
-        <x>
-          <noise type="gaussian">
-            <mean>0.0</mean>
-            <stddev>2e-4</stddev>
-            <bias_mean>0.0000075</bias_mean>
-            <bias_stddev>0.0000008</bias_stddev>
-          </noise>
-        </x>
-        <y>
-          <noise type="gaussian">
-            <mean>0.0</mean>
-            <stddev>2e-4</stddev>
-            <bias_mean>0.0000075</bias_mean>
-            <bias_stddev>0.0000008</bias_stddev>
-          </noise>
-        </y>
-        <z>
-          <noise type="gaussian">
-            <mean>0.0</mean>
-            <stddev>2e-4</stddev>
-            <bias_mean>0.0000075</bias_mean>
-            <bias_stddev>0.0000008</bias_stddev>
-          </noise>
-        </z>
-      </angular_velocity>
-      <linear_acceleration>
-        <x>
-          <noise type="gaussian">
-            <mean>0.0</mean>
-            <stddev>1.7e-2</stddev>
-            <bias_mean>0.1</bias_mean>
-            <bias_stddev>0.001</bias_stddev>
-          </noise>
-        </x>
-        <y>
-          <noise type="gaussian">
-            <mean>0.0</mean>
-            <stddev>1.7e-2</stddev>
-            <bias_mean>0.1</bias_mean>
-            <bias_stddev>0.001</bias_stddev>
-          </noise>
-        </y>
-        <z>
-          <noise type="gaussian">
-            <mean>0.0</mean>
-            <stddev>1.7e-2</stddev>
-            <bias_mean>0.1</bias_mean>
-            <bias_stddev>0.001</bias_stddev>
-          </noise>
-        </z>
-      </linear_acceleration>
-    </imu>
-  </sensor>
-</gazebo>
   </xacro:macro>
 </robot>

File: description/ros2_control/vehicle_system_multi_interface.ros2_control.xacro (robot description, xacro)
@@ -166,13 +166,14 @@
         <state_interface name="position.y"/>
         <state_interface name="position.z"/>
-        <state_interface name="rot.r"/>
-        <state_interface name="rot.p"/>
-        <state_interface name="rot.y"/>
-        <state_interface name="v.x"/>
-        <state_interface name="v.y"/>
-        <state_interface name="v.z"/>
-        <state_interface name="w.r"/>
-        <state_interface name="w.p"/>
-        <state_interface name="w.y"/>
+        <state_interface name="orientation.w"/>
+        <state_interface name="orientation.x"/>
+        <state_interface name="orientation.y"/>
+        <state_interface name="orientation.z"/>
+        <state_interface name="velocity.u"/>
+        <state_interface name="velocity.v"/>
+        <state_interface name="velocity.w"/>
+        <state_interface name="velocity.p"/>
+        <state_interface name="velocity.q"/>
+        <state_interface name="velocity.r"/>
       </sensor>
     </ros2_control>

Commit message: creating world

File: description/blue/xacro/bluerov2_heavy_reach/urdf.xacro (robot description, xacro)
@@ -31,11 +31,4 @@
       </collision>
     </link>
-      <!-- Robot Footprint -->
-    <link name="${prefix}base_footprint" />
-    <joint name="${prefix}base_footprint_joint" type="fixed">
-      <child link="${prefix}base_footprint" />
-      <parent link="${prefix}base_link" />
-      <origin xyz="0.0 0.0 1.0" rpy="0 0 0"/>
-    </joint>
     <!-- Import camera macro -->
     <xacro:include filename="$(find ros2_control_blue_reach_5)/blue/xacro/camera/urdf.xacro" />

File: description/xacro/urdf.xacro (robot description, xacro)
@@ -2,5 +2,18 @@
 <robot xmlns:xacro="http://ros.org/wiki/xacro">
   <xacro:macro name="bluerov2_heavy_alpha_urdf" params="prefix">
+    <!-- Robot world origin -->
+    <link name="world"/>
+    <link name="world_bottom"/>
+    <joint name="world_bottom_joint" type="fixed">
+      <child link="world_bottom" />
+      <parent link="world" />
+      <origin xyz="0.0 0.0 -6.0" rpy="0 0 0"/>
+    </joint>
     <link name="base_link"/>
+    <joint name="world_joint" type="fixed">
+      <child link="base_link" />
+      <parent link="world" />
+      <origin xyz="0.0 0.0 -1.0" rpy="0 0 0"/>
+    </joint>
     <link name="${prefix}manipulator_mount_link">
       <visual>
