Commit message: renamed project

File: description/ros2_control/robot_system_multi_interface.ros2_control.xacro (robot description, xacro)
@@ -6,5 +6,5 @@
       <hardware>
         <xacro:if value="${use_mock_hardware}">
-          <plugin>ros2_control_demo_example_3/RRBotSystemMultiInterfaceHardware</plugin>
+          <plugin>ros2_control_reach_5/RRBotSystemMultiInterfaceHardware</plugin>
           <param name="example_param_hw_start_duration_sec">0.0</param>
           <param name="example_param_hw_stop_duration_sec">3.0</param>
@@ -12,5 +12,5 @@
         </xacro:if>
         <xacro:unless value="${use_mock_hardware}">
-          <plugin>ros2_control_demo_example_3/ReachSystemMultiInterfaceHardware</plugin>
+          <plugin>ros2_control_reach_5/ReachSystemMultiInterfaceHardware</plugin>
           <param name="device">${device}</param>
           <param name="baud_rate">${baud_rate}</param>

File: description/urdf/alpha_5.urdf.xacro (robot description, xacro)
@@ -19,5 +19,5 @@
             <visual>
                 <geometry>
-                    <mesh filename="package://ros2_control_demo_example_3/meshes/M3-INLINE.stl"/>
+                    <mesh filename="package://ros2_control_reach_5/meshes/M3-INLINE.stl"/>
                 </geometry>
                 <origin rpy="0 0 0" xyz="0 0 0"/>
@@ -44,5 +44,5 @@
             <visual>
                 <geometry>
-                    <mesh filename="package://ros2_control_demo_example_3/meshes/M2-1-1.stl"/>
+                    <mesh filename="package://ros2_control_reach_5/meshes/M2-1-1.stl"/>
                 </geometry>
                 <origin rpy="0 0 0" xyz="0 0 0"/>
@@ -71,5 +71,5 @@
             <visual>
                 <geometry>
-                    <mesh filename="package://ros2_control_demo_example_3/meshes/M2.stl"/>
+                    <mesh filename="package://ros2_control_reach_5/meshes/M2.stl"/>
                 </geometry>
                 <origin rpy="0 0 0" xyz="0 0 0"/>
@@ -110,5 +110,5 @@
             <visual>
                 <geometry>
-                    <mesh filename="package://ros2_control_demo_example_3/meshes/M2-1-3.stl"/>
+                    <mesh filename="package://ros2_control_reach_5/meshes/M2-1-3.stl"/>
                 </geometry>
                 <origin rpy="0 0 0" xyz="0 0 0"/>
@@ -137,5 +137,5 @@
             <visual>
                 <geometry>
-                    <mesh filename="package://ros2_control_demo_example_3/meshes/RS1-100-101-123.stl"/>
+                    <mesh filename="package://ros2_control_reach_5/meshes/RS1-100-101-123.stl"/>
                 </geometry>
                 <origin rpy="0 -1.5707 0" xyz="0 0 0"/>
@@ -174,5 +174,5 @@
             <limit effort="10" lower="0" upper="0.015" velocity="10"/>
         </joint>
-        <xacro:include filename="$(find ros2_control_demo_example_3)/urdf/end_effectors/standard_jaws.urdf.xacro"/>
+        <xacro:include filename="$(find ros2_control_reach_5)/urdf/end_effectors/standard_jaws.urdf.xacro"/>
         <xacro:alpha_standard_jaws parent="${name}_jaws_base_link" name="${name}_standard_jaws" axis_a="${name}_axis_a">
             <origin xyz="0 0 0" rpy="0 0 0"/>

File: description/urdf/end_effectors/standard_jaws.urdf.xacro (robot description, xacro)
@@ -14,5 +14,5 @@
             <visual>
                 <geometry>
-                    <mesh filename="package://ros2_control_demo_example_3/meshes/end_effectors/RS1-124.stl"/>
+                    <mesh filename="package://ros2_control_reach_5/meshes/end_effectors/RS1-124.stl"/>
                 </geometry>
                 <material name="${name}_black"/>
@@ -22,5 +22,5 @@
             <visual>
                 <geometry>
-                    <mesh filename="package://ros2_control_demo_example_3/meshes/end_effectors/RS1-130.stl"/>
+                    <mesh filename="package://ros2_control_reach_5/meshes/end_effectors/RS1-130.stl"/>
                 </geometry>
                 <material name="${name}_black"/>
@@ -45,5 +45,5 @@
             <visual>
                 <geometry>
-                    <mesh filename="package://ros2_control_demo_example_3/meshes/end_effectors/RS1-139.stl"/>
+                    <mesh filename="package://ros2_control_reach_5/meshes/end_effectors/RS1-139.stl"/>
                 </geometry>
                 <material name="${name}_black"/>

File: description/urdf/robot_system_multi_interface.urdf.xacro (robot description, xacro)
@@ -13,7 +13,7 @@
   <xacro:arg name="baud_rate" default="115200"/>
   <!-- Import RRBot macro -->
-  <xacro:include filename="$(find ros2_control_demo_example_3)/urdf/alpha_5.urdf.xacro"/>
+  <xacro:include filename="$(find ros2_control_reach_5)/urdf/alpha_5.urdf.xacro"/>
   <!-- Import RRBot ros2_control description -->
-  <xacro:include filename="$(find ros2_control_demo_example_3)/ros2_control/robot_system_multi_interface.ros2_control.xacro" />
+  <xacro:include filename="$(find ros2_control_reach_5)/ros2_control/robot_system_multi_interface.ros2_control.xacro" />
   <!-- Used for fixing robot -->
   <link name="base_link"/>

Commit message: added casadi dep

File: description/ros2_control/robot_system_multi_interface.ros2_control.xacro (robot description, xacro)
@@ -10,4 +10,6 @@
           <param name="example_param_hw_stop_duration_sec">3.0</param>
           <param name="example_param_hw_slowdown">${slowdown}</param>
+          <param name="serial_port">${serial_port}</param>
+          <param name="state_update_frequency">${state_update_frequency}</param>
         </xacro:if>
         <xacro:unless value="${use_mock_hardware}">

File: description/xacro/urdf.xacro (robot description, xacro)
@@ -59,5 +59,5 @@
     </link>
     <joint name="${prefix}manipulator_mount_joint" type="fixed">
-      <origin rpy="0 0 0" xyz="0.24 -0.099 0.029" />
+      <origin rpy="0 0 0" xyz="0.14 0.0 -0.12" />
       <parent link="${prefix}base_link" />
       <child link="${prefix}manipulator_mount_link" />

Commit message: clean up

File: description/ros2_control/robot_system_multi_interface.ros2_control.xacro (robot description, xacro)
@@ -2,13 +2,9 @@
 <robot xmlns:xacro="http://www.ros.org/wiki/xacro">
   <xacro:macro name="robot_system_multi_interface"
-  params="name prefix serial_port state_update_frequency use_mock_hardware slowdown">
+  params="name prefix serial_port state_update_frequency use_mock_hardware">
     <ros2_control name="${name}" type="system">
       <hardware>
         <xacro:if value="${use_mock_hardware}">
           <plugin>ros2_control_blue_reach_5/RRBotSystemMultiInterfaceHardware</plugin>
-          <param name="example_param_hw_start_duration_sec">0.0</param>
-          <param name="example_param_hw_stop_duration_sec">3.0</param>
-          <param name="example_param_hw_slowdown">${slowdown}</param>
-          <param name="serial_port">${serial_port}</param>
           <param name="state_update_frequency">${state_update_frequency}</param>
         </xacro:if>

File: description/ros2_control/vehicle_system_multi_interface.ros2_control.xacro (robot description, xacro)
@@ -2,18 +2,12 @@
 <robot xmlns:xacro="http://www.ros.org/wiki/xacro">
   <xacro:macro name="vehicle_system_multi_interface"
-  params="name prefix serial_port state_update_frequency use_mock_hardware slowdown">
+  params="name prefix serial_port state_update_frequency use_mock_hardware">
     <ros2_control name="${name}" type="system">
       <hardware>
         <xacro:if value="${use_mock_hardware}">
           <plugin>ros2_control_blue_reach_5/VehicleSystemMultiInterfaceHardware</plugin>
-          <param name="example_param_hw_start_duration_sec">0.0</param>
-          <param name="example_param_hw_stop_duration_sec">3.0</param>
-          <param name="example_param_hw_slowdown">${slowdown}</param>
         </xacro:if>
         <xacro:unless value="${use_mock_hardware}">
           <plugin>ros2_control_blue_reach_5/VehicleSystemMultiInterfaceHardware</plugin>
-          <param name="example_param_hw_start_duration_sec">0.0</param>
-          <param name="example_param_hw_stop_duration_sec">3.0</param>
-          <param name="example_param_hw_slowdown">${slowdown}</param>
         </xacro:unless>
       </hardware>

File: description/xacro/robot_system_multi_interface.urdf.xacro (robot description, xacro)
@@ -4,5 +4,4 @@
   <xacro:arg name="use_mock_hardware" default="false" />
   <xacro:arg name="prefix" default="alpha" />
-  <xacro:arg name="slowdown" default="100.0" />
   <xacro:arg name="serial_port" default="/dev/ttyUSB0"/>
   <xacro:arg name="state_update_frequency" default="250"/>
@@ -24,6 +23,5 @@
     serial_port="$(arg serial_port)"
     state_update_frequency="$(arg state_update_frequency)"
-    use_mock_hardware="$(arg use_mock_hardware)"
-    slowdown="$(arg slowdown)" />
+    use_mock_hardware="$(arg use_mock_hardware)"/>
   <xacro:vehicle_system_multi_interface
     name="BlueSystemMultiInterface"
@@ -31,5 +29,4 @@
     serial_port="$(arg serial_port)"
     state_update_frequency="$(arg state_update_frequency)"
-    use_mock_hardware="$(arg use_mock_hardware)"
-    slowdown="$(arg slowdown)" />
+    use_mock_hardware="$(arg use_mock_hardware)"/>
 </robot>

File: description/xacro/urdf.xacro (robot description, xacro)
@@ -22,5 +22,5 @@
       <child link="base_link" />
       <parent link="world" />
-      <origin xyz="0.0 0.0 -2.0" rpy="0 0 0"/>
+      <origin xyz="0.0 0.0 -1.0" rpy="0 0 0"/>
     </joint>
     <link name="${prefix}manipulator_mount_link">
